File: TinkerFET.kicad_sch (KiCad schematic)
At the start: 66 parts, among them J1 B+, J2 GND, J3 M+, J4 M-, J5 U262-161N-4BVC11, J6 HOP, J7 ETU, Q1 FDMC8010, Q2 FDMC8010, Q3 DMP32D4SFB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

Commit message: Updated topside capacitors for easier manual assembly
Parts:
- C14, C15: value 100n -> 1u; LCSC Part C307331 -> C52923
Changed lines of the file:
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@@
       (effects (font (size 1.27 1.27)) (justify left))
     )
-    (property "Value" "100n" (at 204.343 96.139 0)
+    (property "Value" "1u" (at 204.343 96.139 0)
       (effects (font (size 1.27 1.27)) (justify left))
     )
@@
       (effects (font (size 1.27 1.27)) hide)
     )
-    (property "LCSC Part" "C307331" (at 203.2 99.06 0)
+    (property "LCSC Part" "C52923" (at 203.2 99.06 0)
       (effects (font (size 1.27 1.27)) hide)
     )
@@
       (effects (font (size 1.27 1.27)) (justify left))
     )
-    (property "Value" "100n" (at 265.811 90.043 0)
+    (property "Value" "1u" (at 265.811 90.043 0)
       (effects (font (size 1.27 1.27)) (justify left))
     )
@@
       (effects (font (size 1.27 1.27)) hide)
     )
-    (property "LCSC Part" "C307331" (at 262.89 88.9 0)
-      (effects (font (size 1.27 1.27)) hide)
-    )
+    (property "LCSC Part" "C52923" (at 262.89 88.9 0)
+      (effects (font (size 1.27 1.27)) hide)
+    )

Commit message: Updated tracer logic level supply FET part
Parts:
- Q3: value DMP32D4SFB -> DMP2165UW; footprint Package_DFN_QFN:Diodes_DFN1006-3 -> Package_TO_SOT_SMD:SOT-323_SC-70; LCSC Part C3282096 -> C388477
Changed lines of the file:
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@@
   (title_block
     (title "TinkerFET Electronics v0.3")
-    (date "2023-05-19")
+    (date "2023-05-30")
     (rev "0.3")
     (comment 2 "by @timchpi")
@@
       (effects (font (size 1.27 1.27)) (justify left))
     )
-    (property "Value" "DMP32D4SFB" (at 165.1 172.085 0)
+    (property "Value" "DMP2165UW" (at 165.1 172.085 0)
       (effects (font (size 1.27 1.27)) (justify left))
     )
-    (property "Footprint" "Package_DFN_QFN:Diodes_DFN1006-3" (at 163.83 176.53 0)
+    (property "Footprint" "Package_TO_SOT_SMD:SOT-323_SC-70" (at 163.83 176.53 0)
       (effects (font (size 1.27 1.27)) hide)
     )
-    (property "Datasheet" "https://www.diodes.com/assets/Datasheets/DMP32D4SFB.pdf" (at 158.75 173.99 0)
+    (property "Datasheet" "https://datasheet.lcsc.com/lcsc/1912111437_Diodes-Incorporated-DMP2165UW-7_C388477.pdf" (at 158.75 173.99 0)
       (effects (font (size 1.27 1.27)) hide)
     )
-    (property "LCSC Part" "C3282096" (at 158.75 173.99 0)
+    (property "LCSC Part" "C388477" (at 158.75 173.99 0)
       (effects (font (size 1.27 1.27)) hide)
     )

Commit message: Updated front side components
To reduce number of different parts needed
Parts:
- C14, C15, C7: value 1u -> 100n; LCSC Part C52923 -> C307331
- R6: value 1k -> 10k; LCSC Part C11702 -> C25744
Other:
- note removed: "Need: VREF for empty mag detection 3V3 Controlled GND A13, GPIO A14, GPIO for tracer, SHDN on OpAmp A15, GPIO for empty mag detection, with low pass, cap on GPIO pin 12V"
Changed lines of the file:
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@@
     (stroke (width 0) (type default))
   )
-  (text "Need:\nVREF for empty mag detection\n3V3 Controlled\nGND\nA13, GPIO\nA14, GPIO for tracer, SHDN on OpAmp\nA15, GPIO for empty mag detection, with low pass, cap on GPIO pin\n12V"
-    (at 295.91 129.54 0)
-    (effects (font (size 1.27 1.27)) (justify left bottom))
-  )
   (text "PWCWAQ2012F-2R2KTT\nCMCW2012F2R2KTT" (at 90.17 26.67 0)
     (effects (font (size 1.27 1.27)) (justify left bottom))
@@
       (effects (font (size 1.27 1.27)) (justify left))
     )
-    (property "Value" "1u" (at 204.343 96.139 0)
+    (property "Value" "100n" (at 204.343 96.139 0)
       (effects (font (size 1.27 1.27)) (justify left))
     )
@@
       (effects (font (size 1.27 1.27)) hide)
     )
-    (property "LCSC Part" "C52923" (at 203.2 99.06 0)
+    (property "LCSC Part" "C307331" (at 203.2 99.06 0)
       (effects (font (size 1.27 1.27)) hide)
     )
@@
       (effects (font (size 1.27 1.27)) (justify right))
     )
-    (property "Value" "1k" (at 257.683 80.772 0)
+    (property "Value" "10k" (at 257.683 80.772 0)
       (effects (font (size 1.27 1.27)) (justify right))
     )
@@
       (effects (font (size 1.27 1.27)) hide)
     )
-    (property "LCSC Part" "C11702" (at 256.54 82.55 0)
+    (property "LCSC Part" "C25744" (at 256.54 82.55 0)
       (effects (font (size 1.27 1.27)) hide)
     )
@@
       (effects (font (size 1.27 1.27)) (justify left))
     )
-    (property "Value" "1u" (at 265.811 90.043 0)
+    (property "Value" "100n" (at 265.811 90.043 0)
       (effects (font (size 1.27 1.27)) (justify left))
     )
@@
       (effects (font (size 1.27 1.27)) hide)
     )
-    (property "LCSC Part" "C52923" (at 262.89 88.9 0)
+    (property "LCSC Part" "C307331" (at 262.89 88.9 0)
       (effects (font (size 1.27 1.27)) hide)
     )
@@
       (effects (font (size 1.27 1.27)) (justify left))
     )
-    (property "Value" "1u" (at 264.541 37.973 0)
+    (property "Value" "100n" (at 264.541 37.973 0)
       (effects (font (size 1.27 1.27)) (justify left))
     )
@@
       (effects (font (size 1.27 1.27)) hide)
     )
-    (property "LCSC Part" "C52923" (at 261.62 36.83 0)
-      (effects (font (size 1.27 1.27)) hide)
-    )
+    (property "LCSC Part" "C307331" (at 261.62 36.83 0)
+      (effects (font (size 1.27 1.27)) hide)
+    )

Commit message: Corrected schematic comment
Other:
- note added: "1/4.3"
- note added: "Designed for 2s > 7.0V 3s < 13.05V"
- note added: "Fuse: 3557-2"
- note removed: "1/6.6"
- note removed: "Designed for 2s > 7.2V 3s < 13.05V"
- note removed: "Fuse: Cased such as 3557-2 Recommanded"
Changed lines of the file:
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@@
   (title_block
     (title "TinkerFET Electronics v0.3")
-    (date "2023-05-30")
+    (date "2023-06-11")
     (rev "0.3")
     (comment 2 "by @timchpi")
@@
     (effects (font (size 1.27 1.27)) (justify left bottom))
   )
-  (text "1/6.6" (at 255.27 33.02 0)
+  (text "1/4.3" (at 255.27 33.02 0)
     (effects (font (size 1.27 1.27)) (justify left bottom))
   )
-  (text "Fuse:\nCased such as\n3557-2\nRecommanded" (at 209.55 52.07 0)
+  (text "Fuse:\n3557-2" (at 190.5 26.67 0)
     (effects (font (size 1.27 1.27)) (justify left bottom))
   )
-  (text "Designed for\n2s > 7.2V\n3s < 13.05V" (at 153.67 31.75 0)
+  (text "Designed for\n2s > 7.0V\n3s < 13.05V" (at 153.67 31.75 0)
     (effects (font (size 1.27 1.27)) (justify left bottom))
   )
